File: VIO-Board.kicad_sch (KiCad schematic)
At the start: 4 parts

Commit message: workin...
Parts:
- removed R?: (no value), symbol Device:R_US
- removed R?: 27, Resistor_SMD:R_0402_1005Metric, symbol Device:R_US
- removed U?: (no value), symbol FT234XD:FT234XD
- added C? (x2): 4u7, Capacitor_SMD:C_0402_1005Metric, symbol Device:C
- added C? (x2): 100n, Capacitor_SMD:C_0402_1005Metric, symbol Device:C
- added R?: (no value), symbol Device:R_US
- added U?: CP2102N-Axx-xQFN28, Package_DFN_QFN:QFN-28-1EP_5x5mm_P0.5mm_EP3.35x3.35mm, symbol Interface_USB:CP2102N-Axx-xQFN28
- J?: value (none) -> USB_B_Micro; footprint (none) -> Connector_USB:USB_Micro-B_Molex_47346-0001
Connections:
- net GNDREF: now also C?.2, C?.2, C?.2, C?.2, U?.29 (GND), U?.3 (GND)
- net VBUS: now also C?.1, C?.1, U?.7 (VREGIN), U?.8 (VBUS)
- net D+: now reaches J?.3 (D+)
- net D+: now also U?.4 (D+)
- net D-: now reaches J?.2 (D-)
- net D-: now also U?.5 (D-)
- new net: R?.2, U?.9 (~{RST})
- new net +3V3: C?.1, C?.1, R?.1, U?.6 (VDD)
- new net RX: U?.25 (RXD)
- new net TX: U?.26 (TXD)
- no-connect marks 1 -> 19

Commit message: add led again
Parts:
- added D?: (no value), symbol Device:LED
- added R?: (no value), symbol Device:R_US
- R?: value (none) -> 5k1; footprint (none) -> Resistor_SMD:R_0402_1005Metric
Connections:
- net +3V3: now also D?.2 (A)
- net GNDREF: now also R?.1
- new net: D?.1 (K), R?.2
Changed lines of the file:
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@@
+    (stroke (width 0) (type default) (color 0 0 0 0))
+  )
+  (wire (pts (xy 163.83 38.1) (xy 173.99 38.1))
     (stroke (width 0) (type default) (color 0 0 0 0))
   )
@@
     (stroke (width 0) (type default) (color 0 0 0 0))
   )
+  (wire (pts (xy 181.61 38.1) (xy 185.42 38.1))
+    (stroke (width 0) (type default) (color 0 0 0 0))
+  )
+  (wire (pts (xy 185.42 30.48) (xy 185.42 38.1))
+    (stroke (width 0) (type default) (color 0 0 0 0))
+  )
   (wire (pts (xy 143.51 30.48) (xy 137.16 30.48))
     (stroke (width 0) (type default) (color 0 0 0 0))
   )
+  (wire (pts (xy 163.83 31.75) (xy 163.83 30.48))
+    (stroke (width 0) (type default) (color 0 0 0 0))
+  )
   (wire (pts (xy 91.44 80.01) (xy 86.36 80.01))
     (stroke (width 0) (type default) (color 0 0 0 0))
@@
     (stroke (width 0) (type default) (color 0 0 0 0))
   )
+  (wire (pts (xy 163.83 30.48) (xy 173.99 30.48))
+    (stroke (width 0) (type default) (color 0 0 0 0))
+  )
+  (wire (pts (xy 170.18 31.75) (xy 163.83 31.75))
+    (stroke (width 0) (type default) (color 0 0 0 0))
+  )
   (wire (pts (xy 158.75 48.26) (xy 163.83 48.26))
+    (stroke (width 0) (type default) (color 0 0 0 0))
+  )
+  (wire (pts (xy 185.42 30.48) (xy 181.61 30.48))
     (stroke (width 0) (type default) (color 0 0 0 0))
   )
@@
   (label "D-" (at 91.44 80.01 180)
     (effects (font (size 1.27 1.27)) (justify right bottom))
+  )
+  (symbol (lib_id "Device:R_US") (at 177.8 38.1 90) (unit 1)
+    (in_bom yes) (on_board yes)
+    (property "Reference" "R?" (id 0) (at 177.8 34.29 90))
+    (property "Value" "" (id 1) (at 177.8 36.83 90))
+    (property "Footprint" "" (id 2) (at 178.054 37.084 90)
+      (effects (font (size 1.27 1.27)) hide)
+    )
+    (property "Datasheet" "https://www.mouser.com/datasheet/2/315/AOA0000C301-1488782.pdf" (id 3) (at 177.8 38.1 0)
+      (effects (font (size 1.27 1.27)) hide)
+    )
+    (property "Mouser" "https://www.mouser.com/ProductDetail/Panasonic/ERJ-2GEJ221X?qs=sGAEpiMZZMvdGkrng054t8AJgcdMkx7xHJFSutAlOIQ%3D" (id 4) (at 177.8 38.1 90)
+      (effects (font (size 1.27 1.27)) hide)
+    )
+    (pin "1")
+    (pin "2")
   )
   (symbol (lib_id "Device:C") (at 163.83 34.29 0) (unit 1)
@@
     (pin "1")
   )
+  (symbol (lib_id "Device:LED") (at 177.8 30.48 180) (unit 1)
+    (in_bom yes) (on_board yes) (fields_autoplaced)
+    (property "Reference" "D?" (id 0) (at 179.3875 22.86 0))
+    (property "Value" "" (id 1) (at 179.3875 25.4 0))
+    (property "Footprint" "" (id 2) (at 177.8 30.48 0)
+      (effects (font (size 1.27 1.27)) hide)
+    )
+    (property "Datasheet" "~" (id 3) (at 177.8 30.48 0)
+      (effects (font (size 1.27 1.27)) hide)
+    )
+    (property "Mouser" "https://www.mouser.com/ProductDetail/ROHM-Semiconductor/SML-D12V1WT86?qs=M3jcYzEJUdEt%252Bt18c0BExg%3D%3D" (id 4) (at 177.8 30.48 90)
+      (effects (font (size 1.27 1.27)) hide)
+    )
+    (pin "1")
+    (pin "2")
+  )
   (symbol (lib_id "Device:C") (at 137.16 34.29 0) (unit 1)
     (in_bom yes) (on_board yes) (fields_autoplaced)
@@
       (effects (font (size 1.27 1.27)) (justify left))
     )
-    (property "Value" "" (id 1) (at 114.3 45.7199 0)
-      (effects (font (size 1.27 1.27)) (justify left))
-    )
-    (property "Footprint" "" (id 2) (at 112.776 44.704 90)
+    (property "Value" "5k1" (id 1) (at 114.3 45.7199 0)
+      (effects (font (size 1.27 1.27)) (justify left))
+    )
+    (property "Footprint" "Resistor_SMD:R_0402_1005Metric" (id 2) (at 112.776 44.704 90)
       (effects (font (size 1.27 1.27)) hide)
     )
@@
       (reference "C?") (unit 1) (value "4u7") (footprint "Capacitor_SMD:C_0402_1005Metric")
     )
+    (path "/a6522efe-efaa-4294-8978-e8c504504a39"
+      (reference "D?") (unit 1) (value "RED") (footprint "LED_SMD:LED_0603_1608Metric")
+    )
     (path "/bed7de3e-af0a-4641-9494-7dcb327ba2a0"
       (reference "J?") (unit 1) (value "USB_B_Micro") (footprint "Connector_USB:USB_Micro-B_Molex_47346-0001")
     )
+    (path "/012a9e13-a0a9-42dd-8736-632b7014e582"
+      (reference "R?") (unit 1) (value "220") (footprint "Resistor_SMD:R_0402_1005Metric")
+    )
     (path "/df1dfced-018d-4945-a3a7-025f4b9800ea"
