File: VIO-Board.kicad_sch (KiCad schematic)
At the start: 7 parts

Commit message: connectors
Parts:
- added J? (x2): (no value), symbol Connector:Conn_01x02_Male
- added J?: (no value), symbol Connector:Conn_01x05_Male
Connections:
- net GNDREF: now also J?.1 (Pin_1), J?.1 (Pin_1), J?.1 (Pin_1)
- net RX: now also J?.3 (Pin_3)
- net TX: now also J?.2 (Pin_2)
- net VBUS: now also J?.5 (Pin_5)
- new net SYNC: J?.2 (Pin_2), J?.2 (Pin_2), J?.4 (Pin_4)
Changed lines of the file:
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@@
   (no_connect (at 158.75 63.5))
   (no_connect (at 158.75 60.96))
+  (wire (pts (xy 191.77 107.95) (xy 198.12 107.95))
+    (stroke (width 0) (type default) (color 0 0 0 0))
+  )
+  (wire (pts (xy 198.12 110.49) (xy 191.77 110.49))
+    (stroke (width 0) (type default) (color 0 0 0 0))
+  )
   (wire (pts (xy 158.75 50.8) (xy 163.83 50.8))
     (stroke (width 0) (type default) (color 0 0 0 0))
   )
+  (wire (pts (xy 191.77 80.01) (xy 198.12 80.01))
+    (stroke (width 0) (type default) (color 0 0 0 0))
+  )
   (wire (pts (xy 151.13 38.1) (xy 163.83 38.1))
     (stroke (width 0) (type default) (color 0 0 0 0))
@@
     (stroke (width 0) (type default) (color 0 0 0 0))
   )
+  (wire (pts (xy 191.77 96.52) (xy 198.12 96.52))
+    (stroke (width 0) (type default) (color 0 0 0 0))
+  )
   (wire (pts (xy 143.51 30.48) (xy 137.16 30.48))
     (stroke (width 0) (type default) (color 0 0 0 0))
   )
+  (wire (pts (xy 191.77 74.93) (xy 198.12 74.93))
+    (stroke (width 0) (type default) (color 0 0 0 0))
+  )
   (wire (pts (xy 91.44 80.01) (xy 86.36 80.01))
     (stroke (width 0) (type default) (color 0 0 0 0))
   )
+  (wire (pts (xy 191.77 77.47) (xy 198.12 77.47))
+    (stroke (width 0) (type default) (color 0 0 0 0))
+  )
   (wire (pts (xy 86.36 77.47) (xy 91.44 77.47))
     (stroke (width 0) (type default) (color 0 0 0 0))
@@
     (stroke (width 0) (type default) (color 0 0 0 0))
   )
+  (wire (pts (xy 198.12 82.55) (xy 191.77 82.55))
+    (stroke (width 0) (type default) (color 0 0 0 0))
+  )
   (wire (pts (xy 111.76 48.26) (xy 133.35 48.26))
     (stroke (width 0) (type default) (color 0 0 0 0))
@@
     (stroke (width 0) (type default) (color 0 0 0 0))
   )
+  (wire (pts (xy 198.12 72.39) (xy 191.77 72.39))
+    (stroke (width 0) (type default) (color 0 0 0 0))
+  )
+  (wire (pts (xy 191.77 93.98) (xy 198.12 93.98))
+    (stroke (width 0) (type default) (color 0 0 0 0))
+  )
   (wire (pts (xy 88.9 72.39) (xy 86.36 72.39))
     (stroke (width 0) (type default) (color 0 0 0 0))
@@
     (effects (font (size 1.27 1.27)) (justify right bottom))
   )
+  (label "TX" (at 198.12 80.01 180)
+    (effects (font (size 1.27 1.27)) (justify right bottom))
+  )
   (label "D+" (at 91.44 77.47 180)
+    (effects (font (size 1.27 1.27)) (justify right bottom))
+  )
+  (label "SYNC" (at 198.12 93.98 180)
     (effects (font (size 1.27 1.27)) (justify right bottom))
   )
@@
     (effects (font (size 1.27 1.27)) (justify left bottom))
   )
+  (label "SYNC" (at 198.12 107.95 180)
+    (effects (font (size 1.27 1.27)) (justify right bottom))
+  )
   (label "TX" (at 163.83 48.26 180)
+    (effects (font (size 1.27 1.27)) (justify right bottom))
+  )
+  (label "SYNC" (at 198.12 74.93 180)
     (effects (font (size 1.27 1.27)) (justify right bottom))
   )
@@
     (effects (font (size 1.27 1.27)) (justify right bottom))
   )
+  (label "RX" (at 198.12 77.47 180)
+    (effects (font (size 1.27 1.27)) (justify right bottom))
+  )
+  (symbol (lib_id "Connector:Conn_01x02_Male") (at 186.69 96.52 0) (mirror x) (unit 1)
+    (in_bom yes) (on_board yes) (fields_autoplaced)
+    (property "Reference" "J?" (id 0) (at 185.42 93.9799 0)
+      (effects (font (size 1.27 1.27)) (justify right))
+    )
+    (property "Value" "" (id 1) (at 185.42 96.5199 0)
+      (effects (font (size 1.27 1.27)) (justify right))
+    )
+    (property "Footprint" "" (id 2) (at 186.69 96.52 0)
+      (effects (font (size 1.27 1.27)) hide)
+    )
+    (property "Datasheet" "~" (id 3) (at 186.69 96.52 0)
+      (effects (font (size 1.27 1.27)) hide)
+    )
+    (pin "1")
+    (pin "2")
+  )
   (symbol (lib_id "Device:C") (at 163.83 34.29 0) (unit 1)
     (in_bom yes) (on_board yes) (fields_autoplaced)
@@
     (pin "1")
     (pin "2")
+  )
+  (symbol (lib_id "power:VBUS") (at 198.12 72.39 0) (unit 1)
+    (in_bom yes) (on_board yes) (fields_autoplaced)
+    (property "Reference" "#PWR?" (id 0) (at 198.12 76.2 0)
+      (effects (font (size 1.27 1.27)) hide)
+    )
+    (property "Value" "VBUS" (id 1) (at 198.12 67.31 0))
+    (property "Footprint" "" (id 2) (at 198.12 72.39 0)
+      (effects (font (size 1.27 1.27)) hide)
+    )
+    (property "Datasheet" "" (id 3) (at 198.12 72.39 0)
+      (effects (font (size 1.27 1.27)) hide)
+    )
+    (pin "1")
+  )
+  (symbol (lib_id "power:GNDREF") (at 198.12 82.55 0) (unit 1)
+    (in_bom yes) (on_board yes)
+    (property "Reference" "#PWR?" (id 0) (at 198.12 88.9 0)
+      (effects (font (size 1.27 1.27)) hide)
+    )
+    (property "Value" "" (id 1) (at 198.12 87.63 0))
+    (property "Footprint" "" (id 2) (at 198.12 82.55 0)
+      (effects (font (size 1.27 1.27)) hide)
+    )
+    (property "Datasheet" "" (id 3) (at 198.12 82.55 0)
+      (effects (font (size 1.27 1.27)) hide)
+    )
+    (pin "1")
+  )
+  (symbol (lib_id "power:GNDREF") (at 198.12 96.52 0) (unit 1)
+    (in_bom yes) (on_board yes)
+    (property "Reference" "#PWR?" (id 0) (at 198.12 102.87 0)
+      (effects (font (size 1.27 1.27)) hide)
+    )
+    (property "Value" "GNDREF" (id 1) (at 194.31 101.6 0)
+      (effects (font (size 1.27 1.27)) (justify left))
+    )
+    (property "Footprint" "" (id 2) (at 198.12 96.52 0)
+      (effects (font (size 1.27 1.27)) hide)
+    )
+    (property "Datasheet" "" (id 3) (at 198.12 96.52 0)
+      (effects (font (size 1.27 1.27)) hide)
+    )
+    (pin "1")
   )
   (symbol (lib_id "power:+3V3") (at 163.83 30.48 0) (unit 1)
@@
     (pin "1")
   )
+  (symbol (lib_id "Connector:Conn_01x05_Male") (at 186.69 77.47 0) (mirror x) (unit 1)
+    (in_bom yes) (on_board yes) (fields_autoplaced)
+    (property "Reference" "J?" (id 0) (at 187.325 87.63 0))
+    (property "Value" "" (id 1) (at 187.325 85.09 0))
+    (property "Footprint" "" (id 2) (at 186.69 77.47 0)
+      (effects (font (size 1.27 1.27)) hide)
+    )
+    (property "Datasheet" "~" (id 3) (at 186.69 77.47 0)
+      (effects (font (size 1.27 1.27)) hide)
+    )
+    (pin "1")
+    (pin "2")
+    (pin "3")
+    (pin "4")
+    (pin "5")
+  )
   (symbol (lib_id "power:GNDREF") (at 124.46 38.1 0) (unit 1)
     (in_bom yes) (on_board yes) (fields_autoplaced)
@@
     (pin "2")
   )
+  (symbol (lib_id "power:GNDREF") (at 198.12 110.49 0) (unit 1)
+    (in_bom yes) (on_board yes)
+    (property "Reference" "#PWR?" (id 0) (at 198.12 116.84 0)
+      (effects (font (size 1.27 1.27)) hide)
+    )
+    (property "Value" "GNDREF" (id 1) (at 194.31 115.57 0)
+      (effects (font (size 1.27 1.27)) (justify left))
+    )
+    (property "Footprint" "" (id 2) (at 198.12 110.49 0)
+      (effects (font (size 1.27 1.27)) hide)
+    )
+    (property "Datasheet" "" (id 3) (at 198.12 110.49 0)
+      (effects (font (size 1.27 1.27)) hide)
+    )
+    (pin "1")
+  )
   (symbol (lib_id "power:+3V3") (at 111.76 40.64 0) (unit 1)
     (in_bom yes) (on_board yes) (fields_autoplaced)
@@
     (pin "2")
   )
+  (symbol (lib_id "Connector:Conn_01x02_Male") (at 186.69 110.49 0) (mirror x) (unit 1)
+    (in_bom yes) (on_board yes) (fields_autoplaced)
+    (property "Reference" "J?" (id 0) (at 185.42 107.9499 0)
+      (effects (font (size 1.27 1.27)) (justify right))
+    )
+    (property "Value" "" (id 1) (at 185.42 110.4899 0)
+      (effects (font (size 1.27 1.27)) (justify right))
+    )
+    (property "Footprint" "" (id 2) (at 186.69 110.49 0)
+      (effects (font (size 1.27 1.27)) hide)
+    )
+    (property "Datasheet" "~" (id 3) (at 186.69 110.49 0)
+      (effects (font (size 1.27 1.27)) hide)
+    )
+    (pin "1")
+    (pin "2")
+  )
   (sheet_instances
     (path "/" (page "1"))
   )
   (symbol_instances
+    (path "/6182b37d-58f2-46f3-845e-68975fb99ac0"
+      (reference "#PWR?") (unit 1) (value "VBUS") (footprint "")
+    )
+    (path "/63db50a8-08b3-4e4d-9454-b7387e6550f0"
+      (reference "#PWR?") (unit 1) (value "GNDREF") (footprint "")
+    )
+    (path "/64d7f1df-eb62-414e-a3d1-ad461f6098b7"
+      (reference "#PWR?") (unit 1) (value "GNDREF") (footprint "")
+    )
     (path "/6632dfaa-9ffe-4983-8f63-a437db3aa83c"
       (reference "#PWR?") (unit 1) (value "+3V3") (footprint "")
@@
       (reference "#PWR?") (unit 1) (value "VBUS") (footprint "")
     )
+    (path "/e7d0015f-945d-4113-843f-b2e06b7c140a"
+      (reference "#PWR?") (unit 1) (value "GNDREF") (footprint "")
+    )
     (path "/e8fd0535-6a40-4369-b4e1-2f7332303594"
       (reference "#PWR?") (unit 1) (value "+3V3") (footprint "")
@@
       (reference "C?") (unit 1) (value "4u7") (footprint "Capacitor_SMD:C_0402_1005Metric")
     )
+    (path "/2809d02f-edcf-4dfb-bf00-37b7a303a65a"
+      (reference "J?") (unit 1) (value "Cam 1") (footprint "Connector_Wire:SolderWire-0.1sqmm_1x02_P3.6mm_D0.4mm_OD1mm")
+    )
     (path "/bed7de3e-af0a-4641-9494-7dcb327ba2a0"
       (reference "J?") (unit 1) (value "USB_B_Micro") (footprint "Connector_USB:USB_Micro-B_Molex_47346-0001")
     )
+    (path "/c5b05bf3-8fc1-4d1a-9f6d-bc237ff10dcf"
+      (reference "J?") (unit 1) (value "IMU") (footprint "Connector_Wire:SolderWire-0.1sqmm_1x05_P3.6mm_D0.4mm_OD1mm")
+    )
+    (path "/f94802d7-b31d-4d1a-be98-fc6a42c4b2a4"
+      (reference "J?") (unit 1) (value "Cam 2") (footprint "Connector_Wire:SolderWire-0.1sqmm_1x02_P3.6mm_D0.4mm_OD1mm")
+    )
     (path "/df1dfced-018d-4945-a3a7-025f4b9800ea"

Commit message: ...
Parts:
- removed J? (x2): (no value), symbol Connector:Conn_01x02_Male
- removed J?: (no value), symbol Connector:Conn_01x05_Male
- added J1: (no value), symbol Connector:Conn_01x02_Female
- added J3: (no value), symbol Connector:Conn_01x09_Male
- added J4, J5: Conn_01x09_Male, Connector_PinHeader_2.54mm:PinHeader_1x09_P2.54mm_Vertical, symbol Connector:Conn_01x09_Male
- added J6: (no value), symbol Connector:Conn_01x09_Female
- added J7, J8: Conn_01x09_Female, Connector_PinSocket_2.54mm:PinSocket_1x09_P2.54mm_Vertical, symbol Connector:Conn_01x09_Female
- R1: renamed from R?; value (none) -> 5k1; footprint (none) -> Resistor_SMD:R_0402_1005Metric
- gave numbers to parts that had none: 6
Connections:
- net GNDREF: now also J1.2 (Pin_2), J3.2 (Pin_2), J3.6 (Pin_6), J4.2 (Pin_2), J4.6 (Pin_6), J5.5 (Pin_5), J6.2 (Pin_2), J6.6 (Pin_6), J7.2 (Pin_2), J7.6 (Pin_6), J8.5 (Pin_5)
- net SYNC: now also J3.5 (Pin_5), J4.5 (Pin_5), J5.4 (Pin_4), J6.5 (Pin_5), J7.5 (Pin_5), J8.4 (Pin_4)
- net VBUS: now also J5.1 (Pin_1), J8.1 (Pin_1)
- net RX renamed RX2
- net RX2: now also J5.9 (Pin_9), J8.9 (Pin_9)
- net TX renamed TX2
- net TX2: now also J5.8 (Pin_8), J8.8 (Pin_8)
- new net 3V3_CAM1: J3.3 (Pin_3), J6.3 (Pin_3)
- new net 3V3_CAM2: J4.3 (Pin_3), J7.3 (Pin_3)
- new net GPIO3/TX_CAM1: J3.4 (Pin_4), J6.4 (Pin_4)
- new net GPIO3/TX_CAM2: J4.4 (Pin_4), J7.4 (Pin_4)
- new net OPTO_GND_CAM1: J3.7 (Pin_7), J6.7 (Pin_7)
- new net OPTO_GND_CAM2: J4.7 (Pin_7), J7.7 (Pin_7)
- new net OPTO_IN_CAM1: J3.9 (Pin_9), J6.9 (Pin_9)
- new net OPTO_IN_CAM2: J4.9 (Pin_9), J7.9 (Pin_9)
- new net OPTO_OUT_CAM1: J3.8 (Pin_8), J6.8 (Pin_8)
- new net OPTO_OUT_CAM2: J4.8 (Pin_8), J7.8 (Pin_8)
- new net RESTORE: J5.6 (Pin_6), J8.6 (Pin_6)
- new net RX1: J5.3 (Pin_3), J8.3 (Pin_3)
- new net SYNC_IN: J5.7 (Pin_7), J8.7 (Pin_7)
- new net TX1: J5.2 (Pin_2), J8.2 (Pin_2)
- new net VS: J1.1 (Pin_1), J3.1 (Pin_1), J4.1 (Pin_1), J6.1 (Pin_1), J7.1 (Pin_1)
Other:
- note added: "CP2102"
- note added: "GPIO2/RX_CAM1"
- note added: "GPIO2/RX_CAM2"
- note added: "Headers"
- note added: "POWER"
- note added: "SYNC_OUT"
- note added: "USB"
- moved on the sheet: C1, C2, C3, C4, J2, R1, U1
