File: VIO-Board.kicad_sch (KiCad schematic)
At the start: 17 parts, among them J1 Conn_01x02_Female, J2 USB_B_Micro, J3 Conn_01x09_Male, J4 Conn_01x09_Male, J5 Conn_01x09_Male, J6 Conn_01x09_Female, J7 Conn_01x09_Female, J8 Conn_01x09_Female

Commit message: final touches
Parts:
- J2: value USB_B_Micro -> (none); footprint Connector_USB:USB_Micro-B_Molex_47346-0001 -> (none); Mouser (none) -> https://www.mouser.com/ProductDetail/Molex/47346-0001?qs=c2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
- U1: renamed from U?; Mouser (none) -> https://www.mouser.com/ProductDetail/Silicon-Labs/CP2102N-A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
- gave numbers to parts that had none: 3
Changed lines of the file:
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@@
   (symbol (lib_id "power:GNDREF") (at 80.01 66.04 0) (unit 1)
     (in_bom yes) (on_board yes)
-    (property "Reference" "#PWR?" (id 0) (at 80.01 72.39 0)
+    (property "Reference" "#PWR09" (id 0) (at 80.01 72.39 0)
       (effects (font (size 1.27 1.27)) hide)
     )
@@
   (symbol (lib_id "Device:R_US") (at 76.2 66.04 90) (unit 1)
     (in_bom yes) (on_board yes) (fields_autoplaced)
-    (property "Reference" "R?" (id 0) (at 76.2 59.69 90))
+    (property "Reference" "R3" (id 0) (at 76.2 59.69 90))
     (property "Value" "" (id 1) (at 76.2 62.23 90))
     (property "Footprint" "" (id 2) (at 76.454 65.024 90)
@@
   (symbol (lib_id "Device:R_US") (at 68.58 66.04 90) (unit 1)
     (in_bom yes) (on_board yes) (fields_autoplaced)
-    (property "Reference" "R?" (id 0) (at 68.58 59.69 90))
+    (property "Reference" "R2" (id 0) (at 68.58 59.69 90))
     (property "Value" "" (id 1) (at 68.58 62.23 90))
     (property "Footprint" "" (id 2) (at 68.834 65.024 90)
@@
   (symbol (lib_id "power:GNDREF") (at 78.74 88.9 0) (unit 1)
     (in_bom yes) (on_board yes) (fields_autoplaced)
-    (property "Reference" "#PWR?" (id 0) (at 78.74 95.25 0)
+    (property "Reference" "#PWR08" (id 0) (at 78.74 95.25 0)
       (effects (font (size 1.27 1.27)) hide)
     )
@@
   (symbol (lib_id "power:+3V3") (at 116.84 40.64 0) (unit 1)
     (in_bom yes) (on_board yes) (fields_autoplaced)
-    (property "Reference" "#PWR09" (id 0) (at 116.84 44.45 0)
+    (property "Reference" "#PWR011" (id 0) (at 116.84 44.45 0)
       (effects (font (size 1.27 1.27)) hide)
     )
@@
   (symbol (lib_id "Interface_USB:CP2102N-Axx-xQFN20") (at 99.06 81.28 0) (unit 1)
     (in_bom yes) (on_board yes) (fields_autoplaced)
-    (property "Reference" "U?" (id 0) (at 101.0794 109.22 0)
+    (property "Reference" "U1" (id 0) (at 101.0794 109.22 0)
       (effects (font (size 1.27 1.27)) (justify left))
     )
@@
     )
     (property "Datasheet" "https://www.silabs.com/documents/public/data-sheets/cp2102n-datasheet.pdf" (id 3) (at 100.33 100.33 0)
+      (effects (font (size 1.27 1.27)) hide)
+    )
+    (property "Mouser" "https://www.mouser.com/ProductDetail/Silicon-Labs/CP2102N-A02-GQFN20?qs=u16ybLDytRaG8WdlP0fT2g%3D%3D" (id 4) (at 99.06 81.28 0)
       (effects (font (size 1.27 1.27)) hide)
     )
@@
   (symbol (lib_id "power:VBUS") (at 77.47 40.64 0) (unit 1)
     (in_bom yes) (on_board yes) (fields_autoplaced)
-    (property "Reference" "#PWR05" (id 0) (at 77.47 44.45 0)
+    (property "Reference" "#PWR06" (id 0) (at 77.47 44.45 0)
       (effects (font (size 1.27 1.27)) hide)
     )
@@
     (in_bom yes) (on_board yes) (fields_autoplaced)
     (property "Reference" "J2" (id 0) (at 34.29 35.56 0))
-    (property "Value" "USB_B_Micro" (id 1) (at 34.29 38.1 0))
-    (property "Footprint" "Connector_USB:USB_Micro-B_Molex_47346-0001" (id 2) (at 38.1 49.53 0)
+    (property "Value" "" (id 1) (at 34.29 38.1 0))
+    (property "Footprint" "" (id 2) (at 38.1 49.53 0)
       (effects (font (size 1.27 1.27)) hide)
     )
@@
       (effects (font (size 1.27 1.27)) hide)
     )
+    (property "Mouser" "https://www.mouser.com/ProductDetail/Molex/47346-0001?qs=c2CV6XM0DweJBWaSeyWeCw%3D%3D" (id 4) (at 34.29 48.26 0)
+      (effects (font (size 1.27 1.27)) hide)
+    )
     (pin "1")
     (pin "2")
@@
   (symbol (lib_id "power:GNDREF") (at 99.06 109.22 0) (unit 1)
     (in_bom yes) (on_board yes) (fields_autoplaced)
-    (property "Reference" "#PWR08" (id 0) (at 99.06 115.57 0)
+    (property "Reference" "#PWR010" (id 0) (at 99.06 115.57 0)
       (effects (font (size 1.27 1.27)) hide)
     )
@@
   (symbol (lib_id "power:GNDREF") (at 116.84 48.26 0) (unit 1)
     (in_bom yes) (on_board yes) (fields_autoplaced)
-    (property "Reference" "#PWR010" (id 0) (at 116.84 54.61 0)
+    (property "Reference" "#PWR012" (id 0) (at 116.84 54.61 0)
       (effects (font (size 1.27 1.27)) hide)
     )
@@
   (symbol (lib_id "power:GNDREF") (at 77.47 48.26 0) (unit 1)
     (in_bom yes) (on_board yes) (fields_autoplaced)
-    (property "Reference" "#PWR06" (id 0) (at 77.47 54.61 0)
+    (property "Reference" "#PWR07" (id 0) (at 77.47 54.61 0)
       (effects (font (size 1.27 1.27)) hide)
     )
@@
   (symbol (lib_id "power:VBUS") (at 60.96 66.04 0) (unit 1)
     (in_bom yes) (on_board yes) (fields_autoplaced)
-    (property "Reference" "#PWR07" (id 0) (at 60.96 69.85 0)
+    (property "Reference" "#PWR04" (id 0) (at 60.96 69.85 0)
       (effects (font (size 1.27 1.27)) hide)
     )
@@
   (symbol (lib_id "power:+3V3") (at 64.77 50.8 0) (unit 1)
     (in_bom yes) (on_board yes) (fields_autoplaced)
-    (property "Reference" "#PWR04" (id 0) (at 64.77 54.61 0)
+    (property "Reference" "#PWR05" (id 0) (at 64.77 54.61 0)
       (effects (font (size 1.27 1.27)) hide)
     )
@@
   (symbol (lib_id "Power_Protection:SP0503BAHT") (at 67.31 83.82 0) (unit 1)
     (in_bom yes) (on_board yes)
-    (property "Reference" "D?" (id 0) (at 73.66 82.55 0)
+    (property "Reference" "D1" (id 0) (at 73.66 82.55 0)
       (effects (font (size 1.27 1.27)) (justify left))
     )
@@
       (reference "#PWR03") (unit 1) (value "VBUS") (footprint "")
     )
+    (path "/d9d6439f-9b67-4965-963f-2ec0d20a1f84"
+      (reference "#PWR04") (unit 1) (value "VBUS") (footprint "")
+    )
     (path "/e8fd0535-6a40-4369-b4e1-2f7332303594"
-      (reference "#PWR04") (unit 1) (value "+3V3") (footprint "")
+      (reference "#PWR05") (unit 1) (value "+3V3") (footprint "")
     )
     (path "/aaf6d173-f17c-46f4-85ef-8a56f1d078fc"
-      (reference "#PWR05") (unit 1) (value "VBUS") (footprint "")
+      (reference "#PWR06") (unit 1) (value "VBUS") (footprint "")
     )
     (path "/ccbecf91-8464-4655-a9f1-1e717fd2d32f"
-      (reference "#PWR06") (unit 1) (value "GNDREF") (footprint "")
-    )
-    (path "/d9d6439f-9b67-4965-963f-2ec0d20a1f84"
-      (reference "#PWR07") (unit 1) (value "VBUS") (footprint "")
+      (reference "#PWR07") (unit 1) (value "GNDREF") (footprint "")
+    )
+    (path "/56e1cf0e-d61b-4dfe-8d76-cf4629de505d"
+      (reference "#PWR08") (unit 1) (value "GNDREF") (footprint "")
+    )
+    (path "/1085a35a-4fad-41d9-9ca7-e49a6bbaf11c"
+      (reference "#PWR09") (unit 1) (value "GNDREF") (footprint "")
     )
     (path "/bfc19f53-0a87-4bd5-bc60-b8db527a9d57"
-      (reference "#PWR08") (unit 1) (value "GNDREF") (footprint "")
+      (reference "#PWR010") (unit 1) (value "GNDREF") (footprint "")
     )
     (path "/6632dfaa-9ffe-4983-8f63-a437db3aa83c"
-      (reference "#PWR09") (unit 1) (value "+3V3") (footprint "")
+      (reference "#PWR011") (unit 1) (value "+3V3") (footprint "")
     )
     (path "/c088b075-78e4-4c54-8067-d972c3672dc3"
-      (reference "#PWR010") (unit 1) (value "GNDREF") (footprint "")
-    )
-    (path "/1085a35a-4fad-41d9-9ca7-e49a6bbaf11c"
-      (reference "#PWR?") (unit 1) (value "GNDREF") (footprint "")
-    )
-    (path "/56e1cf0e-d61b-4dfe-8d76-cf4629de505d"
-      (reference "#PWR?") (unit 1) (value "GNDREF") (footprint "")
+      (reference "#PWR012") (unit 1) (value "GNDREF") (footprint "")
     )
     (path "/f7a02a4d-5b2a-4743-beba-bffcf39ae8d4"
@@
     )
     (path "/fcb23687-79e7-494b-b78d-610b9b788477"
-      (reference "D?") (unit 1) (value "SP0503BAHT") (footprint "Package_TO_SOT_SMD:SOT-143")
+      (reference "D1") (unit 1) (value "SP0503BAHT") (footprint "Package_TO_SOT_SMD:SOT-143")
     )
     (path "/38b69a3f-9f2a-4119-861c-51e9020433d6"
@@
       (reference "R1") (unit 1) (value "5k1") (footprint "Resistor_SMD:R_0402_1005Metric")
     )
+    (path "/2ff395ea-5491-46d8-9fe0-ef3e45cdd157"
+      (reference "R2") (unit 1) (value "22k1") (footprint "Resistor_SMD:R_0402_1005Metric")
+    )
     (path "/2773960a-b220-4367-b86f-1f2693b6238b"
-      (reference "R?") (unit 1) (value "47k5") (footprint "Resistor_SMD:R_0402_1005Metric")
-    )
-    (path "/2ff395ea-5491-46d8-9fe0-ef3e45cdd157"
-      (reference "R?") (unit 1) (value "22k1") (footprint "Resistor_SMD:R_0402_1005Metric")
+      (reference "R3") (unit 1) (value "47k5") (footprint "Resistor_SMD:R_0402_1005Metric")
     )
     (path "/8c087470-e370-4fb0-9ba5-a82293a7d292"
-      (reference "U?") (unit 1) (value "CP2102N-Axx-xQFN20") (footprint "Package_DFN_QFN:SiliconLabs_QFN-20-1EP_3x3mm_P0.5mm")
-    )
-  )
+      (reference "U1") (unit 1) (value "CP2102N-Axx-xQFN20") (footprint "Package_DFN_QFN:SiliconLabs_QFN-20-1EP_3x3mm_P0.5mm_EP1.8x1.8mm")
+    )
+  )

Commit message: BOM and corrections
Parts:
- R1: value 5k1 -> (none); footprint Resistor_SMD:R_0402_1005Metric -> (none); Mouser https://www.reddit.com/r/tumblr/comments/ujkope/butter_rect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 -> https://www.mouser.com/ProductDetail/Panasonic/ERJ-2RKF5101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
Changed lines of the file:
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@@
       (effects (font (size 1.27 1.27)) (justify left))
     )
-    (property "Value" "5k1" (id 1) (at 67.31 55.8799 0)
+    (property "Value" "" (id 1) (at 67.31 55.8799 0)
       (effects (font (size 1.27 1.27)) (justify left))
     )
-    (property "Footprint" "Resistor_SMD:R_0402_1005Metric" (id 2) (at 65.786 54.864 90)
+    (property "Footprint" "" (id 2) (at 65.786 54.864 90)
       (effects (font (size 1.27 1.27)) hide)
     )
@@
       (effects (font (size 1.27 1.27)) hide)
     )
-    (property "Mouser" "https://www.reddit.com/r/tumblr/comments/ujkope/butter_rectangular_prism/" (id 4) (at 64.77 54.61 90)
+    (property "Mouser" "https://www.mouser.com/ProductDetail/Panasonic/ERJ-2RKF5101X?qs=sGAEpiMZZMvdGkrng054t8AJgcdMkx7xIXmurKOGv8o%3D" (id 4) (at 64.77 54.61 90)
       (effects (font (size 1.27 1.27)) hide)
     )

Commit message: v2.0
Parts:
- added D2: GREEN, LED_SMD:LED_0603_1608Metric, symbol Device:LED
- added D3: RED, LED_SMD:LED_0603_1608Metric, symbol Device:LED
- added JP1, JP2: SolderJumper_2_Open, Jumper:SolderJumper-2_P1.3mm_Open_RoundedPad1.0x1.5mm, symbol Jumper:SolderJumper_2_Open
- added R4: 400, Resistor_SMD:R_0402_1005Metric, symbol Device:R_US
- added R5: 2k, Resistor_SMD:R_0402_1005Metric, symbol Device:R_US
- D1: value (none) -> SP0503BAHT; footprint (none) -> Package_TO_SOT_SMD:SOT-143
- J2: value (none) -> USB_B_Micro; footprint (none) -> Connector_USB:USB_Micro-B_Molex_47346-0001
- R1: value (none) -> 5k1; footprint (none) -> Resistor_SMD:R_0402_1005Metric
- R2: value (none) -> 22k1; footprint (none) -> Resistor_SMD:R_0402_1005Metric
- R3: value (none) -> 47k5; footprint (none) -> Resistor_SMD:R_0402_1005Metric
- U1: value (none) -> CP2102N-Axx-xQFN20; footprint (none) -> Package_DFN_QFN:SiliconLabs_QFN-20-1EP_3x3mm_P0.5mm_EP1.8x1.8mm
Connections:
- net GNDREF: now also J1.1 (Pin_1), D2.1 (K), D3.1 (K), JP1.2 (B); no longer J1.2 (Pin_2)
- net RESTORE: now also JP1.1 (A)
- net RX2: now also U1.18 (TXD); no longer U1.17 (RXD)
- net SYNC: now also JP2.2 (B)
- net SYNC_IN: now also JP2.1 (A)
- net TX2: now also U1.17 (RXD); no longer U1.18 (TXD)
- net VBUS: now also R4.1
- net VS: now also J1.2 (Pin_2), R5.1; no longer J1.1 (Pin_1)
- new net: D3.2 (A), R5.2
- new net: D2.2 (A), R4.2
Other:
- note added: "JUMPERS"
- note added: "LEDs"
