File: VIO-Board-rounded.kicad_pcb (KiCad board)
At the start: 4 copper layers, 39.6 x 39.6 mm, 24 parts, among them J1 Conn_01x02_Female, J2 USB_B_Micro, J3 Conn_01x09_Male, J4 Conn_01x09_Male, J5 Conn_01x09_Male, J6 Conn_01x09_Female, J7 Conn_01x09_Female, J8 Conn_01x09_Female, U1 CP2102N-Axx-xQFN20

Commit message: v2.0
Parts:
- added D2: GREEN, LED_SMD:LED_0603_1608Metric, F.Cu at (79.2, 59.9)
- added D3: RED, LED_SMD:LED_0603_1608Metric, F.Cu at (79.2, 61.7)
- added JP1: SolderJumper_2_Open, Jumper:SolderJumper-2_P1.3mm_Open_RoundedPad1.0x1.5mm, B.Cu at (77.7, 81.3)
- added JP2: SolderJumper_2_Open, Jumper:SolderJumper-2_P1.3mm_Open_RoundedPad1.0x1.5mm, B.Cu at (77.7, 78.2)
- added R4: 400, Resistor_SMD:R_0402_1005Metric, F.Cu at (75.4, 59.9)
- added R5: 2k, Resistor_SMD:R_0402_1005Metric, F.Cu at (79.0, 63.2)
- moved G*** 2.79 mm to (76.5, 70.1)
Connections:
- J1 pad 1: /VS -> GNDREF
- J1 pad 2: GNDREF -> VS
- J3 pad 1: /VS -> VS
- J4 pad 1: /VS -> VS
- J6 pad 1: /VS -> VS
- J7 pad 1: /VS -> VS
- U1 pad 17: /RX2 -> /TX2
- U1 pad 18: /TX2 -> /RX2
Routing:
- net /SYNC_IN: track 3.53 -> 12.3 mm
- net /SYNC: track 62.0 -> 70.8 mm
- net VS: track 0.00 -> 6.86 mm, vias 0 -> 1
- net GNDREF: track 14.9 -> 20.6 mm, vias 14 -> 16
- net /RESTORE: track 3.53 -> 7.30 mm
- net Net-(D2-Pad2): track 0.00 -> 2.51 mm
- net Net-(D3-Pad2): track 0.00 -> 1.53 mm
- net /RX2: track 36.5 -> 35.0 mm
- added copper zone on B.Cu, net VS
- removed copper zone on B.Cu, net /VS
Other:
- board text added: "EXT"
- board text added: "RSTR BRIDGE"
- board text added: "SYNC BRIDGE"
- board text added: "USB"
